File: Quads_MCU_PCB/Quads_MCU_PCB.kicad_pcb (KiCad board)
At the start: 4 copper layers, 100 x 100 mm, 108 parts, among them J1 USB_C_Receptacle_USB2.0_16P, J2 Conn_01x06_Pin, J3 Conn_01x02_Pin, J4 Conn_01x04_Pin, J5 Conn_01x04_Pin, J6 Conn_01x04_Pin, J7 Conn_01x04_Pin, SW1 SW_Push, U1 STM32H723ZGTx, U10 BMI088, U3 ADM3057ExRW, U4 TSR_1-2450, U5 AP7361C-33E, U6 ADM3057ExRW, U7 ADM3057ExRW, U8 MCP2518FD-xQBB, U9 ADM3057ExRW, Y1 40MHz, Y2 25MHz

Commit message: Layout: General positions
Parts:
- moved J6 94.9 mm to (130.4, 64.5), turned to 90 degrees
- moved J5 81.8 mm to (130.7, 90.8), turned to 90 degrees
- moved U7 72.7 mm to (50.6, 80.6), turned to 180 degrees
- moved U9 62.4 mm to (61.1, 107.2), turned to 180 degrees
- moved J2 53.9 mm to (96.6, 42.0), turned to -90 degrees
- moved C1 53.2 mm to (44.3, 122.2)
- moved C10 53.2 mm to (47.1, 122.2)
- moved C11 53.2 mm to (47.1, 124.1)
- moved C12 53.2 mm to (47.1, 126.1)
- moved C13 53.2 mm to (47.1, 128.1)
- moved C14 53.2 mm to (47.1, 130.0)
- moved C15 53.2 mm to (47.1, 132.0)
- moved C16 53.2 mm to (47.1, 134.0)
- moved C17 53.2 mm to (47.1, 135.9)
- moved C18 53.2 mm to (50.0, 122.2)
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Routing:
- net Net-(C2-Pad2): track 0.00 -> 1.50 mm
- net GND: track 0.00 -> 0.79 mm, vias 0 -> 1
